File: IEEE_PCB_1/IEEE_PCB_1.kicad_pcb (KiCad board)
At the start: 2 copper layers, 53.8 x 123.2 mm, 0 parts

Commit message: Added Outlines to Library
Other:
- board outline removed
Changed lines of the file:
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@@
   (general
     (thickness 1.6)
-    (drawings 74)
+    (drawings 0)
     (tracks 0)
     (zones 0)
@@
     (uvia_drill 0.1)
   )
-  (dimension 125.73 (width 0.15) (layer Dwgs.User)
-    (gr_text "125.730 mm" (at 141 113.665 270) (layer Dwgs.User)
-      (effects (font (size 1 1) (thickness 0.15)))
-    )
-    (feature1 (pts (xy 102.87 176.53) (xy 140.286421 176.53)))
-    (feature2 (pts (xy 102.87 50.8) (xy 140.286421 50.8)))
-    (crossbar (pts (xy 139.7 50.8) (xy 139.7 176.53)))
-    (arrow1a (pts (xy 139.7 176.53) (xy 139.113579 175.403496)))
-    (arrow1b (pts (xy 139.7 176.53) (xy 140.286421 175.403496)))
-    (arrow2a (pts (xy 139.7 50.8) (xy 139.113579 51.926504)))
-    (arrow2b (pts (xy 139.7 50.8) (xy 140.286421 51.926504)))
-  )
-  (gr_line (start 147.71523 86.871269) (end 147.228178 84.310849) (layer Edge.Cuts) (width 0.072))
-  (gr_line (start 148.061683 89.287636) (end 147.71523 86.871269) (layer Edge.Cuts) (width 0.072))
-  (gr_line (start 148.43598 92.845761) (end 148.061683 89.287636) (layer Edge.Cuts) (width 0.072))
-  (gr_arc (start 139.544585 95.516047) (end 141.606182 103.054318) (angle -18.23305911) (layer Edge.Cuts) (width 0.072))
-  (gr_arc (start 138.814866 93.735596) (end 148.440406 94.576208) (angle -10.27518122) (layer Edge.Cuts) (width 0.072))
-  (gr_arc (start 143.20842 94.119286) (end 148.12337 95.970154) (angle -15.6442186) (layer Edge.Cuts) (width 0.072))
-  (gr_line (start 113.636217 162.676443) (end 113.775687 153.413613) (layer Edge.Cuts) (width 0.072))
-  (gr_arc (start 122.191021 88.313551) (end 127.524896 85.565986) (angle -21.00316086) (layer Edge.Cuts) (width 0.072))
-  (gr_arc (start 121.022318 87.389334) (end 122.359246 81.998667) (angle -16.71556144) (layer Edge.Cuts) (width 0.072))
-  (gr_arc (start 120.99822 86.894241) (end 120.752286 81.841925) (angle -17.68547945) (layer Edge.Cuts) (width 0.072))
-  (gr_line (start 113.799999 127.762432) (end 113.850407 98.038377) (layer Edge.Cuts) (width 0.072))
-  (gr_line (start 113.8 63.499234) (end 109.724609 65.397958) (layer Edge.Cuts) (width 0.072))
-  (gr_arc (start 104.519221 165.574355) (end 100.07834 174.27503) (angle -29.36752832) (layer Edge.Cuts) (width 0.072))
-  (gr_line (start 113.8 57.990448) (end 113.8 63.499234) (layer Edge.Cuts) (width 0.072))
-  (gr_line (start 94.866446 155.008149) (end 95.040731 164.116294) (layer Edge.Cuts) (width 0.072))
-  (gr_line (start 94.737717 128.092236) (end 94.866446 155.008149) (layer Edge.Cuts) (width 0.072))
-  (gr_arc (start 120.383753 88.276532) (end 109.724609 65.397958) (angle -13.67309135) (layer Edge.Cuts) (width 0.072))
-  (gr_line (start 113.84195 55.814456) (end 113.8 57.990448) (layer Edge.Cuts) (width 0.072))
-  (gr_line (start 113.329483 167.672483) (end 113.636217 162.676443) (layer Edge.Cuts) (width 0.072))
-  (gr_arc (start 129.252494 88.863736) (end 147.316027 97.825874) (angle -5.752662909) (layer Edge.Cuts) (width 0.072))
-  (gr_arc (start 137.834408 93.121614) (end 146.624667 99.017588) (angle -7.463230018) (layer Edge.Cuts) (width 0.072))
-  (gr_arc (start 133.589812 90.274602) (end 145.717081 100.238367) (angle -5.555227283) (layer Edge.Cuts) (width 0.072))
-  (gr_arc (start 121.230418 89.335093) (end 104.618607 68.565959) (angle -13.14708787) (layer Edge.Cuts) (width 0.072))
-  (gr_arc (start 138.999049 93.626647) (end 136.407757 103.054775) (angle -15.37319395) (layer Edge.Cuts) (width 0.072))
-  (gr_arc (start 108.919328 86.693546) (end 95.207211 83.846924) (angle -10.73761612) (layer Edge.Cuts) (width 0.072))
-  (gr_arc (start 105.7215 166.951981) (end 112.599946 170.281773) (angle -20.42123129) (layer Edge.Cuts) (width 0.072))
-  (gr_line (start 113.850407 98.038377) (end 114.216137 89.687867) (layer Edge.Cuts) (width 0.072))
-  (gr_arc (start 134.394457 90.93573) (end 144.744216 101.309897) (angle -5.661046493) (layer Edge.Cuts) (width 0.072))
-  (gr_arc (start 120.718105 89.142952) (end 97.123853 78.090128) (angle -13.37299204) (layer Edge.Cuts) (width 0.072))
-  (gr_line (start 94.703952 109.870101) (end 94.737717 128.092236) (layer Edge.Cuts) (width 0.072))
-  (gr_line (start 129.1884 92.174627) (end 129.86981 95.998157) (layer Edge.Cuts) (width 0.072))
-  (gr_line (start 95.040731 164.116294) (end 95.355863 168.934943) (layer Edge.Cuts) (width 0.072))
-  (gr_arc (start 126.848452 90.75336) (end 115.283335 85.561181) (angle -19.35648615) (layer Edge.Cuts) (width 0.072))
-  (gr_line (start 94.916942 86.451494) (end 94.776229 96.539402) (layer Edge.Cuts) (width 0.072))
-  (gr_line (start 113.97176 54.003563) (end 113.84195 55.814456) (layer Edge.Cuts) (width 0.072))
-  (gr_arc (start 122.606848 91.203085) (end 119.229058 82.155418) (angle -10.8999738) (layer Edge.Cuts) (width 0.072))
-  (gr_line (start 114.154629 52.57248) (end 113.97176 54.003563) (layer Edge.Cuts) (width 0.072))
-  (gr_arc (start 138.379084 95.882346) (end 134.193898 102.031662) (angle -18.8708034) (layer Edge.Cuts) (width 0.072))
-  (gr_arc (start 105.247354 164.147801) (end 96.137073 170.950906) (angle -26.20934446) (layer Edge.Cuts) (width 0.072))
-  (gr_line (start 128.466914 88.163961) (end 129.1884 92.174627) (layer Edge.Cuts) (width 0.072))
-  (gr_arc (start 114.514321 52.626702) (end 114.399143 52.281662) (angle -62.96790617) (layer Edge.Cuts) (width 0.072))
-  (gr_arc (start 137.146483 95.201408) (end 130.746767 98.451245) (angle -18.22645476) (layer Edge.Cuts) (width 0.072))
-  (gr_line (start 94.776229 96.539402) (end 94.703952 109.870101) (layer Edge.Cuts) (width 0.072))
-  (gr_arc (start 139.949212 93.77816) (end 129.86981 95.998157) (angle -14.50074444) (layer Edge.Cuts) (width 0.072))
-  (gr_arc (start 121.380432 89.453183) (end 100.330039 72.888716) (angle -13.0982033) (layer Edge.Cuts) (width 0.072))
-  (gr_arc (start 142.515817 89.804209) (end 132.084318 100.289855) (angle -10.61275344) (layer Edge.Cuts) (width 0.072))
-  (gr_arc (start 140.692821 97.248964) (end 143.86127 102.030795) (angle -11.40412675) (layer Edge.Cuts) (width 0.072))
-  (gr_arc (start 138.999036 93.521247) (end 138.999919 103.404397) (angle -15.29037224) (layer Edge.Cuts) (width 0.072))
-  (gr_arc (start 121.640914 88.930051) (end 126.185736 83.836768) (angle -19.06655378) (layer Edge.Cuts) (width 0.072))
-  (gr_arc (start 120.630516 87.961812) (end 117.579129 82.957372) (angle -34.45001245) (layer Edge.Cuts) (width 0.072))
-  (gr_arc (start 119.178784 94.822744) (end 124.272602 82.631547) (angle -8.747794194) (layer Edge.Cuts) (width 0.072))
-  (gr_arc (start 99.364301 168.54097) (end 95.355863 168.934943) (angle -31.13724214) (layer Edge.Cuts) (width 0.072))
-  (gr_arc (start 117.888176 90.530008) (end 128.466914 88.163961) (angle -14.64637281) (layer Edge.Cuts) (width 0.072))
-  (gr_line (start 113.775687 153.413613) (end 113.799999 127.762432) (layer Edge.Cuts) (width 0.072))
-  (gr_arc (start 104.504206 166.362695) (end 109.451041 173.874619) (angle -30.80263225) (layer Edge.Cuts) (width 0.072))
-  (gr_arc (start 104.554357 166.438859) (end 104.915927 175.334774) (angle -31.03869568) (layer Edge.Cuts) (width 0.072))
-  (gr_arc (start 119.036972 92.092146) (end 139.762778 70.779523) (angle -11.54449274) (layer Edge.Cuts) (width 0.072))
-  (gr_line (start 124.978419 52.461025) (end 120.252323 52.270052) (layer Edge.Cuts) (width 0.072))
-  (gr_arc (start 124.76124 57.196334) (end 126.25 52.695899) (angle -15.67843579) (layer Edge.Cuts) (width 0.072))
-  (gr_arc (start 131.144121 85.947667) (end 146.68314 81.97645) (angle -6.177280518) (layer Edge.Cuts) (width 0.072))
-  (gr_line (start 129.932878 64.541666) (end 127 63.5) (layer Edge.Cuts) (width 0.072))
-  (gr_arc (start 126.080675 53.207758) (end 126.600161 53.063517) (angle -56.17775937) (layer Edge.Cuts) (width 0.072))
-  (gr_arc (start 121.528598 88.204437) (end 135.078217 67.062855) (angle -13.10231513) (layer Edge.Cuts) (width 0.072))
-  (gr_line (start 147.228178 84.310849) (end 146.68314 81.97645) (layer Edge.Cuts) (width 0.072))
-  (gr_arc (start 119.290384 91.831599) (end 143.581903 75.332176) (angle -11.6144439) (layer Edge.Cuts) (width 0.072))
-  (gr_circle (center 120.258547 57.756711) (end 122.711984 57.756711) (layer Edge.Cuts) (width 0.072))
-  (gr_arc (start 115.375322 55.206018) (end 115.455173 52.12407) (angle -19.94366965) (layer Edge.Cuts) (width 0.072))
-  (gr_arc (start 110.79512 56.315341) (end 126.959774 55.782196) (angle -5.839925835) (layer Edge.Cuts) (width 0.072))
-  (gr_line (start 127 58.222) (end 126.959774 55.782196) (layer Edge.Cuts) (width 0.072))
-  (gr_arc (start 118.802904 55.228507) (end 126.821633 54.140217) (angle -7.788996572) (layer Edge.Cuts) (width 0.072))
-  (gr_line (start 120.252323 52.270052) (end 115.455173 52.12407) (layer Edge.Cuts) (width 0.072))
-  (gr_arc (start 124.039643 88.605805) (end 146.165593 80.32743) (angle -13.67217788) (layer Edge.Cuts) (width 0.072))
-  (gr_line (start 127 63.5) (end 127 58.222) (layer Edge.Cuts) (width 0.072))
 )

Commit message: PCB
first pcb ball orientation
Parts:
- added ?: , , F.Cu at (108.0, 51.0)
- added C1: 0.01 uF, Capacitor_THT:CP_Radial_D5.0mm_P2.00mm, F.Cu at (142.5, 108.0)
- added C2: 10 uF, Capacitor_THT:CP_Radial_D5.0mm_P2.00mm, F.Cu at (150.0, 108.0)
- added D1: LED, LED_THT:LED_D5.0mm_Clear, F.Cu at (165.0, 77.0)
- added D2: LED, LED_THT:LED_D5.0mm_Clear, F.Cu at (114.5, 75.0)
- added D3: LED, LED_THT:LED_D5.0mm_Clear, F.Cu at (137.0, 68.5)
- added D4: LED, LED_THT:LED_D5.0mm_Clear, F.Cu at (100.5, 98.5)
- added D5: LED, LED_THT:LED_D5.0mm_Clear, F.Cu at (177.0, 104.0)
- added D6: LED, LED_THT:LED_D5.0mm_Clear, F.Cu at (102.5, 118.0)
- added D7: LED, LED_THT:LED_D5.0mm_Clear, F.Cu at (138.0, 144.5)
- added D8: LED, LED_THT:LED_D5.0mm_Clear, F.Cu at (116.5, 137.0)
- added D9: LED, LED_THT:LED_D5.0mm_Clear, F.Cu at (166.0, 127.5)
- added R1: 1K, Resistor_THT:R_Axial_DIN0309_L9.0mm_D3.2mm_P12.70mm_Horizontal, F.Cu at (146.5, 88.5)
- added RV1: R_POT_US, IEEE_PCB_Ornament:CT6EP504, F.Cu at (155.0, 98.0)
- added U1: 555, IEEE_PCB_Ornament:555, F.Cu at (134.0, 91.0)
- added U2: 4017, IEEE_PCB_Ornament:4017, F.Cu at (121.5, 91.0)
- added U3: EG1218, IEEE_PCB_Ornament:EG1218, F.Cu at (137.5, 117.0)
- added U4: 1058TR, IEEE_PCB_Ornament:1058TR, F.Cu at (137.5, 120.7)
Routing:
- net Net-(D5-Pad2): track 0.00 -> 55.0 mm
- net +3V3: track 0.00 -> 47.5 mm
- net Net-(D1-Pad2): track 0.00 -> 46.8 mm
- net Net-(D7-Pad2): track 0.00 -> 46.1 mm
- net Net-(D9-Pad2): track 0.00 -> 46.1 mm
- net Net-(D8-Pad2): track 0.00 -> 35.4 mm
- net Net-(D3-Pad2): track 0.00 -> 35.1 mm
- net Net-(C2-Pad1): track 0.00 -> 31.4 mm
- net Net-(D6-Pad2): track 0.00 -> 23.3 mm
- net Net-(R1-Pad2): track 0.00 -> 22.9 mm
- net Net-(D2-Pad2): track 0.00 -> 21.2 mm
- net Net-(D4-Pad2): track 0.00 -> 18.5 mm
- net Net-(U2-Pad11): track 0.00 -> 11.1 mm
- net Net-(U3-Pad2): track 0.00 -> 11.0 mm
- net Net-(C1-Pad1): track 0.00 -> 9.74 mm
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- added copper zone on B.Cu, net GND
Other:
- board outline added: 89.3 x 109 mm

Commit message: Rev5
Parts:
- moved U3 21.0 mm to (158.5, 117.0)
- moved C2 7.00 mm to (157.0, 108.0)
- moved C1 6.00 mm to (148.5, 108.0)
Routing:
- net Net-(U3-Pad2): track 11.0 -> 33.2 mm
- net +3V3: track 47.5 -> 68.5 mm
- net Net-(C1-Pad1): track 9.74 -> 13.4 mm
- net Net-(C2-Pad1): track 31.4 -> 33.1 mm
