File: IEEE_PCB_SMD/IEEE_PCB_SMD.sch (KiCad schematic (older format))
At the start: 18 parts, among them U1 555, U2 4017, U3 EG1218, U4 EG1218, U5 1058TR

Commit message: rev
Parts:
- removed U3: EG1218, symbol IEEE_PCB_Ornament:EG1218
Connections:
- net labels added: +3V3
- net labels removed: AllON
- wire segments 110 -> 82
Changed lines of the file:
@@
-$EndComp
-$Comp
-L IEEE_PCB_Ornament:EG1218 U3
-U 1 1 62F9767B
-P 9250 4400
-F 0 "U3" V 9204 4022 50  0000 R CNN
-F 1 "EG1218" V 9295 4022 50  0000 R CNN
-F 2 "" H 9250 4500 50  0001 C CNN
-F 3 "" H 9250 4500 50  0001 C CNN
-	1    9250 4400
-	0    -1   1    0
 $EndComp
 $Comp
@@
 Connection ~ 9000 5450
 $Comp
-L power:+3.3V #PWR0107
-U 1 1 62FB176C
-P 9550 4000
-F 0 "#PWR0107" H 9550 3850 50  0001 C CNN
-F 1 "+3.3V" H 9565 4173 50  0000 C CNN
-F 2 "" H 9550 4000 50  0001 C CNN
-F 3 "" H 9550 4000 50  0001 C CNN
-	1    9550 4000
-	1    0    0    -1
-$EndComp
-Wire Wire Line
-	9550 4000 9550 4100
-Text GLabel 9650 4850 2    50   Output ~ 0
-AllON
-Wire Wire Line
-	9550 4700 9550 4850
-Wire Wire Line
-	9550 4850 9650 4850
-$Comp
 L Device:LED D1
 U 1 1 62FB7653
@@
 	3050 3650 3050 3050
 Wire Wire Line
-	3050 3050 2350 3050
-Wire Wire Line
 	3200 3750 3000 3750
 Wire Wire Line
 	3000 3750 3000 3350
 Wire Wire Line
-	3000 3350 2350 3350
-Wire Wire Line
 	3200 3850 2950 3850
 Wire Wire Line
 	2950 3850 2950 3650
-Wire Wire Line
-	2950 3650 2350 3650
-Wire Wire Line
-	3200 3950 2350 3950
 $Comp
 L power:GND #PWR0108
@@
 Wire Wire Line
 	3900 3550 4200 3550
-Text GLabel 2400 2050 2    50   Input ~ 0
-AllON
-Wire Wire Line
-	2150 2450 2350 2450
-Wire Wire Line
-	2150 2750 2350 2750
-Text GLabel 2400 2350 2    50   Input ~ 0
-AllON
-Text GLabel 2400 2650 2    50   Input ~ 0
-AllON
-Text GLabel 2400 2950 2    50   Input ~ 0
-AllON
-Text GLabel 2400 3250 2    50   Input ~ 0
-AllON
-Text GLabel 2400 3550 2    50   Input ~ 0
-AllON
-Text GLabel 2400 3850 2    50   Input ~ 0
-AllON
-Text GLabel 4200 4250 0    50   Input ~ 0
-AllON
-Text GLabel 4300 3850 0    50   Input ~ 0
-AllON
-Wire Wire Line
-	2400 2350 2350 2350
-Wire Wire Line
-	2350 2350 2350 2450
-Connection ~ 2350 2450
-Wire Wire Line
-	2350 2450 3150 2450
-Wire Wire Line
-	2150 2150 2350 2150
-Wire Wire Line
-	2400 2050 2350 2050
-Wire Wire Line
-	2350 2050 2350 2150
-Connection ~ 2350 2150
-Wire Wire Line
-	2350 2150 3200 2150
-Wire Wire Line
-	2400 2650 2350 2650
-Wire Wire Line
-	2350 2650 2350 2750
-Connection ~ 2350 2750
-Wire Wire Line
-	2350 2750 3100 2750
-Wire Wire Line
-	2400 2950 2350 2950
-Wire Wire Line
-	2350 2950 2350 3050
-Connection ~ 2350 3050
-Wire Wire Line
-	2350 3050 2150 3050
-Wire Wire Line
-	2400 3250 2350 3250
-Wire Wire Line
-	2350 3250 2350 3350
-Connection ~ 2350 3350
-Wire Wire Line
-	2350 3350 2150 3350
-Wire Wire Line
-	2400 3550 2350 3550
-Wire Wire Line
-	2350 3550 2350 3650
-Connection ~ 2350 3650
-Wire Wire Line
-	2350 3650 2150 3650
-Wire Wire Line
-	2400 3850 2350 3850
-Wire Wire Line
-	2350 3850 2350 3950
-Connection ~ 2350 3950
-Wire Wire Line
-	2350 3950 2150 3950
-Wire Wire Line
-	3900 3950 4350 3950
-Wire Wire Line
-	4300 3850 4350 3850
-Wire Wire Line
-	4350 3850 4350 3950
-Connection ~ 4350 3950
-Wire Wire Line
-	4350 3950 4400 3950
-Wire Wire Line
-	4200 4250 4300 4250
-Connection ~ 4300 4250
 Text Notes 550  650  0    100  ~ 0
 LED Circuit
@@
 Text Notes 7100 3550 0    100  ~ 0
 Power
+$Comp
+L power:+3V3 #PWR?
+U 1 1 630C63F7
+P 9200 4400
+F 0 "#PWR?" H 9200 4250 50  0001 C CNN
+F 1 "+3V3" H 9215 4573 50  0000 C CNN
+F 2 "" H 9200 4400 50  0001 C CNN
+F 3 "" H 9200 4400 50  0001 C CNN
+	1    9200 4400
+	1    0    0    -1
+$EndComp
+Wire Wire Line
+	2150 2150 3200 2150
+Wire Wire Line
+	2150 2450 3150 2450
+Wire Wire Line
+	2150 2750 3100 2750
+Wire Wire Line
+	2150 3050 3050 3050
+Wire Wire Line
+	2150 3350 3000 3350
+Wire Wire Line
+	2150 3650 2950 3650
+Wire Wire Line
+	3200 3950 2150 3950
+Wire Wire Line
+	3900 3950 4400 3950
 $EndSCHEMATC

Commit message: SMD Rev2
Parts:
- D1, D2, D3: value LED -> YELLOW
- D4, D5, D6, D7, D8, D9: value LED -> RED
- renumbered U4 to U3, U5 to U4
Connections:
- no-connect marks 1 -> 8
Other:
- moved on the sheet: U2

Commit message: PCB rev smd
Parts:
- C1, C2: footprint (none) -> Capacitor_THT:CP_Radial_D5.0mm_P2.00mm
- D1, D2, D3, D4, D5, D6, D7, D8, D9: footprint (none) -> IEEE_PCB_Ornament:LED_SMD
- R1: footprint (none) -> Resistor_THT:R_Axial_DIN0309_L9.0mm_D3.2mm_P12.70mm_Horizontal
- RV1: footprint (none) -> IEEE_PCB_Ornament:CT6EP504
- U1: footprint (none) -> IEEE_PCB_Ornament:555
- U2: footprint (none) -> IEEE_PCB_Ornament:4017
- U3: footprint (none) -> IEEE_PCB_Ornament:EG1218
- U4: footprint (none) -> IEEE_PCB_Ornament:1058TR
Changed lines of the file:
@@
 F 0 "U1" H 8950 2165 50  0000 C CNN
 F 1 "555" H 8950 2074 50  0000 C CNN
-F 2 "" H 8900 1350 50  0001 C CNN
+F 2 "IEEE_PCB_Ornament:555" H 8900 1350 50  0001 C CNN
 F 3 "" H 8900 1350 50  0001 C CNN
 	1    8900 1800
@@
 F 0 "U2" H 4100 3975 50  0000 C CNN
 F 1 "4017" H 4100 3884 50  0000 C CNN
-F 2 "" H 4150 3450 50  0001 C CNN
+F 2 "IEEE_PCB_Ornament:4017" H 4150 3450 50  0001 C CNN
 F 3 "" H 4150 3450 50  0001 C CNN
 	1    4100 3450
@@
 F 0 "U4" H 8308 5715 50  0000 C CNN
 F 1 "1058TR" H 8308 5624 50  0000 C CNN
-F 2 "" H 8250 5650 50  0001 C CNN
+F 2 "IEEE_PCB_Ornament:1058TR" H 8250 5650 50  0001 C CNN
 F 3 "" H 8250 5650 50  0001 C CNN
 	1    8250 5300
@@
 F 0 "U3" V 8854 4772 50  0000 R CNN
 F 1 "EG1218" V 8945 4772 50  0000 R CNN
-F 2 "" H 8900 5250 50  0001 C CNN
+F 2 "IEEE_PCB_Ornament:EG1218" H 8900 5250 50  0001 C CNN
 F 3 "" H 8900 5250 50  0001 C CNN
 	1    8900 5150
@@
 F 0 "C1" H 9200 2500 50  0000 L CNN
 F 1 "0.01 uF" H 9000 2400 50  0000 L CNN
-F 2 "" H 9400 2450 50  0001 C CNN
+F 2 "Capacitor_THT:CP_Radial_D5.0mm_P2.00mm" H 9400 2450 50  0001 C CNN
 F 3 "~" H 9400 2450 50  0001 C CNN
 	1    9400 2450
@@
 F 0 "C2" H 9841 2496 50  0000 L CNN
 F 1 "10 uF" H 9841 2405 50  0000 L CNN
-F 2 "" H 9750 2450 50  0001 C CNN
+F 2 "Capacitor_THT:CP_Radial_D5.0mm_P2.00mm" H 9750 2450 50  0001 C CNN
 F 3 "~" H 9750 2450 50  0001 C CNN
 	1    9750 2450
@@
 F 0 "RV1" H 10082 2046 50  0000 R CNN
 F 1 "500K" H 10082 1955 50  0000 R CNN
-F 2 "" H 10150 2000 50  0001 C CNN
+F 2 "IEEE_PCB_Ornament:CT6EP504" H 10150 2000 50  0001 C CNN
 F 3 "~" H 10150 2000 50  0001 C CNN
 	1    10150 2000
@@
 F 0 "R1" H 9968 1746 50  0000 L CNN
 F 1 "1k" H 9968 1655 50  0000 L CNN
-F 2 "" H 9900 1700 50  0001 C CNN
+F 2 "Resistor_THT:R_Axial_DIN0309_L9.0mm_D3.2mm_P12.70mm_Horizontal" H 9900 1700 50  0001 C CNN
 F 3 "~" H 9900 1700 50  0001 C CNN
 	1    9900 1700
@@
 F 0 "D1" H 2700 2400 50  0000 C CNN
 F 1 "YELLOW" H 2900 2200 50  0000 C CNN
-F 2 "" H 2800 2300 50  0001 C CNN
+F 2 "IEEE_PCB_Ornament:LED_SMD" H 2800 2300 50  0001 C CNN
 F 3 "~" H 2800 2300 50  0001 C CNN
 	1    2800 2300
@@
 F 0 "D2" H 2700 2700 50  0000 C CNN
 F 1 "YELLOW" H 2900 2500 50  0000 C CNN
-F 2 "" H 2800 2600 50  0001 C CNN
+F 2 "IEEE_PCB_Ornament:LED_SMD" H 2800 2600 50  0001 C CNN
 F 3 "~" H 2800 2600 50  0001 C CNN
 	1    2800 2600
@@
 F 0 "D3" H 2700 3000 50  0000 C CNN
 F 1 "YELLOW" H 2900 2800 50  0000 C CNN
-F 2 "" H 2800 2900 50  0001 C CNN
+F 2 "IEEE_PCB_Ornament:LED_SMD" H 2800 2900 50  0001 C CNN
 F 3 "~" H 2800 2900 50  0001 C CNN
 	1    2800 2900
@@
 F 0 "D4" H 2700 3450 50  0000 C CNN
 F 1 "RED" H 2800 3250 50  0000 C CNN
-F 2 "" H 2800 3350 50  0001 C CNN
+F 2 "IEEE_PCB_Ornament:LED_SMD" H 2800 3350 50  0001 C CNN
 F 3 "~" H 2800 3350 50  0001 C CNN
 	1    2800 3350
@@
 F 0 "D5" H 2700 3750 50  0000 C CNN
 F 1 "RED" H 2800 3550 50  0000 C CNN
-F 2 "" H 2800 3650 50  0001 C CNN
+F 2 "IEEE_PCB_Ornament:LED_SMD" H 2800 3650 50  0001 C CNN
 F 3 "~" H 2800 3650 50  0001 C CNN
 	1    2800 3650
@@
 F 0 "D6" H 2700 4050 50  0000 C CNN
 F 1 "RED" H 2800 3850 50  0000 C CNN
-F 2 "" H 2800 3950 50  0001 C CNN
+F 2 "IEEE_PCB_Ornament:LED_SMD" H 2800 3950 50  0001 C CNN
 F 3 "~" H 2800 3950 50  0001 C CNN
 	1    2800 3950
@@
 F 0 "D7" H 2700 4650 50  0000 C CNN
 F 1 "RED" H 2800 4450 50  0000 C CNN
-F 2 "" H 2800 4550 50  0001 C CNN
+F 2 "IEEE_PCB_Ornament:LED_SMD" H 2800 4550 50  0001 C CNN
 F 3 "~" H 2800 4550 50  0001 C CNN
 	1    2800 4550
@@
 F 0 "D8" H 2700 4950 50  0000 C CNN
 F 1 "RED" H 2800 4750 50  0000 C CNN
-F 2 "" H 2800 4850 50  0001 C CNN
+F 2 "IEEE_PCB_Ornament:LED_SMD" H 2800 4850 50  0001 C CNN
 F 3 "~" H 2800 4850 50  0001 C CNN
 	1    2800 4850
@@
 F 0 "D9" H 2700 5250 50  0000 C CNN
 F 1 "RED" H 2800 5050 50  0000 C CNN
-F 2 "" H 2800 5150 50  0001 C CNN
+F 2 "IEEE_PCB_Ornament:LED_SMD" H 2800 5150 50  0001 C CNN
 F 3 "~" H 2800 5150 50  0001 C CNN
 	1    2800 5150

Commit message: SMD Rev3
Parts:
- removed U4: 1058TR, IEEE_PCB_Ornament:1058TR, symbol IEEE_PCB_Ornament:1058TR
- added D10, D11, D12: D, IEEE_PCB_Ornament:SDM20U40Q, symbol Device:D
- added U4: EG1218, IEEE_PCB_Ornament:EG1218, symbol IEEE_PCB_Ornament:EG1218
- added U5: CR2025TR, IEEE_PCB_Ornament:CR2025TR, symbol IEEE_PCB_Ornament:CR2025TR
- RV1: value 500K -> 100K
Connections:
- net labels added: ALLON
- wire segments 82 -> 101
- no-connect marks 8 -> 9
Other:
- moved on the sheet: D1, D2, D3, D4, D5, D6, D7, D8, D9, U2, U3

Commit message: same
Parts:
- RV1: value 100K -> 50K
Changed lines of the file:
@@
 P 10150 2000
 F 0 "RV1" H 10082 2046 50  0000 R CNN
-F 1 "100K" H 10082 1955 50  0000 R CNN
+F 1 "50K" H 10082 1955 50  0000 R CNN
 F 2 "IEEE_PCB_Ornament:CT6EP504" H 10150 2000 50  0001 C CNN
 F 3 "~" H 10150 2000 50  0001 C CNN
