File: IEEE_DemoTest/IEEE_DemoTest.kicad_sch (KiCad schematic)
At the start: 26 parts, among them SW1 SW_DPDT_x2, U1 LM555xM, U2 4017

Commit message: changed demo
Parts:
- 3V1: renamed from 3V; footprint (none) -> IEEEOrnamentupdate1:CR2025TR
- C1, C2: footprint (none) -> Capacitor_THT:CP_Radial_D5.0mm_P2.00mm
- D1, D2, D3, D4, D5, D6, D7, D8, D9: footprint (none) -> IEEEOrnamentupdate1:IN-S63AT
- R1: footprint (none) -> Resistor_THT:R_Axial_DIN0207_L6.3mm_D2.5mm_P7.62mm_Horizontal
- R10, R2, R3, R4, R5, R6, R7, R8, R9: footprint (none) -> Resistor_SMD:R_0603_1608Metric_Pad0.98x0.95mm_HandSolder
- RV1: footprint (none) -> IEEEOrnamentupdate1:CT6EP504
- SW1: footprint (none) -> IEEEOrnamentupdate1:EG1218
- U2: footprint (none) -> IEEEOrnamentupdate1:4017
